File: PCB/sim800c.sch (EAGLE design)
At the start: 35 parts, among them IC1 ESDA5V3L, IC2 ESDA5V3L, IC3 317EMP, IC4 317EMP, IC5 ESDA5V3L, J1 USB, J2 1, Q1 BC846, Q2 BC846

Commit message: Add files via upload
Parts:
- added C10, C9: (no value), resistor:C-EUC0603
- added R10, R11, R12, R13: (no value), resistor:R-EU_M1206
Connections:
- removed net N$21: C1.+, C2.1, C3.1, D2.C, S1.VBAT, S1.VBAT1
- new net N$19: C9.1, IC3.ADJ, R10.1, R11.2
- new net N$23: R2.2, S1.NETLIGHT
- new net N$24: R1.2, S1.STATUS
- new net N$25: C10.1, IC4.ADJ, R12.1, R13.2
- new net N$28: C5.+, IC4.VO, R12.2
- net +5V: now also C1.+, C2.1, C3.1, D2.C, R10.2, S1.VBAT, S1.VBAT1; no longer C5.+, IC4.VO
- net GND: now also C10.2, C9.2, LED1.K, LED2.K, R11.1, R13.1; no longer IC3.ADJ, IC4.ADJ
- net N$17: now also IC1.1; no longer IC1.2
- net N$18: now also IC1.2; no longer IC1.1
Other:
- moved on the sheet: C4, C5, D1, IC4, LED1, LED2, Q1, Q2, R1, R2, R3, R4

Commit message: Add files via upload
Parts:
- added C11: 100uF, resistor:CPOL-EU140CLH-0810
- added Q3, Q4: BC846, BC846B_215:BC846B,215
- added R14: 0R, resistor:R-EU_M1206
- added R15, R17, R19, R20: 4k7, resistor:R-EU_M1206
- added R16, R18: 47k, resistor:R-EU_M1206
- C6: value (none) -> 1uF
- C7: value (none) -> 100nF
- C8: value (none) -> 22pF
- R5, R6: value (none) -> 22R
- R7, R8, R9: value (none) -> 51R
Connections:
- new net N$1: Q3.E, R16.2, S1.UART2-TXD
- new net N$21: J2.1, R14.1
- new net N$26: C11.+, S1.VRTC
- new net N$27: Q3.B, R15.2, R16.1
- new net N$30: R15.1, R19.1, R20.1, S1.VD-EXT
- new net N$32: Q3.C, R17.2, X3-1.KL
- new net N$34: Q4.B, R19.2
- new net N$35: Q4.C, R20.2, S1.UART2-RXD
- new net N$36: Q4.E, R18.2, X2-2.KL
- net GND: now also C11.-, X2-1.KL
- net N$28: now also R17.1, R18.1, X3-2.KL
- net N$5: now also R14.2; no longer J2.1
Other:
- note added: "GND"
- note added: "Rx"
- note added: "Tx"
- note added: "VDD"
- moved on the sheet: C6, IC5, J1, R5, R6, X2-1, X2-2, X3-1, X3-2

Commit message: Add files via upload
Parts:
- removed D1: 1N4004, diode:1N4004
- removed R4: (no value), resistor:R-EU_M1206
- added R21, R23, R24: 4k7, resistor:R-EU_M1206
- added R22, R25: 47k, resistor:R-EU_M1206
- added X4, X5: (no value), con-wago-500:W237-102
- C4, C5: value (none) -> 470uF; device resistor:CPOL-EU140CLH-0810 -> resistor:CPOL-EU140CLH-1010
- C6: device resistor:CPOL-EU140CLH-0810 -> resistor:CPOL-EU153CLV-0405
- C7: device resistor:CPOL-EU140CLH-0810 -> resistor:C-EUC0805
- C8: device resistor:C-EUC0603 -> resistor:C-EUC0805
- IC3: value 317EMP -> 317T; device linear:317EMP -> linear:317T
- J2: value 1 -> Ant GSM
- R1, R2: value (none) -> 3k3
- R3: value (none) -> 4k7
Connections:
- removed net N$11: S1.UART1_TXD
- new net N$31: Q2.E, R22.1, X4-2.KL
- new net N$33: Q2.B, R3.1
- new net N$38: R22.2, R23.1, X5-2.KL
- new net S$3: Q1.E, R25.1, S1.UART1_TXD
- net GND: now also C7.2, X4-1.KL; no longer C7.-
- net N$12: now also Q2.C, R21.1
- net N$17: now also C7.1; no longer C7.+
- net N$30: now also R21.2, R24.2, R3.2
- net N$8: now also Q1.C, R23.2, X5-1.KL; no longer Q2.C, R3.1
- net N$9: now also Q1.B, R24.1, R25.2; no longer Q1.C, R4.1
Other:
- moved on the sheet: C1, C10, C2, C3, C4, C5, C6, C9, D2, IC3, IC4, LED1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

Commit message: Add files via upload
Connections:
- net N$10: now also IC5.1; no longer IC5.2
- net N$4: now also IC5.2; no longer IC5.1
Changed lines of the file:
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@@
 <pinref part="R5" gate="G$1" pin="1"/>
 <pinref part="J1" gate="G$1" pin="2"/>
-<wire x1="129.54" y1="40.64" x2="132.08" y2="40.64" width="0.1524" layer="91"/>
-<pinref part="IC5" gate="G$1" pin="1"/>
-<wire x1="132.08" y1="40.64" x2="144.78" y2="40.64" width="0.1524" layer="91"/>
+<wire x1="129.54" y1="40.64" x2="144.78" y2="40.64" width="0.1524" layer="91"/>
 <wire x1="144.78" y1="40.64" x2="144.78" y2="33.02" width="0.1524" layer="91"/>
 <wire x1="144.78" y1="33.02" x2="147.32" y2="33.02" width="0.1524" layer="91"/>
-<wire x1="132.08" y1="30.48" x2="132.08" y2="40.64" width="0.1524" layer="91"/>
-<junction x="132.08" y="40.64"/>
+<pinref part="IC5" gate="G$1" pin="2"/>
+<wire x1="129.54" y1="30.48" x2="129.54" y2="40.64" width="0.1524" layer="91"/>
+<junction x="129.54" y="40.64"/>
 </segment>
 </net>
@@
 <pinref part="R6" gate="G$1" pin="1"/>
 <pinref part="J1" gate="G$1" pin="3"/>
-<pinref part="IC5" gate="G$1" pin="2"/>
-<wire x1="129.54" y1="38.1" x2="142.24" y2="38.1" width="0.1524" layer="91"/>
+<wire x1="129.54" y1="38.1" x2="132.08" y2="38.1" width="0.1524" layer="91"/>
+<wire x1="132.08" y1="38.1" x2="142.24" y2="38.1" width="0.1524" layer="91"/>
 <wire x1="142.24" y1="38.1" x2="142.24" y2="30.48" width="0.1524" layer="91"/>
 <wire x1="142.24" y1="30.48" x2="147.32" y2="30.48" width="0.1524" layer="91"/>
-<wire x1="129.54" y1="30.48" x2="129.54" y2="38.1" width="0.1524" layer="91"/>
-<junction x="129.54" y="38.1"/>
+<pinref part="IC5" gate="G$1" pin="1"/>
+<wire x1="132.08" y1="30.48" x2="132.08" y2="38.1" width="0.1524" layer="91"/>
+<junction x="132.08" y="38.1"/>
 </segment>
 </net>
