File: PCB/sim800c.brd (EAGLE design)
At the start: 96.5 x 100 mm, 35 parts, among them IC1 ESDA5V3L, IC2 ESDA5V3L, IC3 317EMP, IC4 317EMP, IC5 ESDA5V3L, J1 USB, J2 1, Q1 BC846, Q2 BC846

Commit message: Add files via upload
Parts:
- added C10, C9: (no value), resistor:C0603
- added R10, R11, R12, R13: (no value), resistor:M1206
- moved R1 60.4 mm to (33.0, 53.3), turned to 270 degrees
- moved LED1 57.0 mm to (33.0, 58.4), turned to 270 degrees
- moved R8 55.7 mm to (41.9, 16.5), turned to 180 degrees
- moved R9 55.7 mm to (41.9, 11.4), turned to 180 degrees
- moved C8 53.1 mm to (52.1, 6.35)
- moved R2 50.0 mm to (38.1, 53.3), turned to 270 degrees
- moved R7 46.2 mm to (41.9, 6.35), turned to 180 degrees
- moved LED2 45.9 mm to (38.1, 58.4), turned to 270 degrees
- moved C7 42.7 mm to (33.0, 29.2), turned to 270 degrees
- moved C2 34.2 mm to (58.4, 52.1), turned to 90 degrees
- moved C3 34.2 mm to (55.9, 52.1), turned to 90 degrees
- moved C1 16.2 mm to (45.7, 55.9)
- moved C5 15.3 mm to (41.9, 76.2)
- moved D2 13.7 mm to (52.1, 55.9)
- moved C4 5.24 mm to (41.9, 91.4)
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Connections:
- removed net N$21: C1.+, C2.1, C3.1, D2.C, S1.34, S1.35
- new net N$19: C9.1, IC3.1, R10.1, R11.2
- new net N$23: R2.2, S1.41
- new net N$24: R1.2, S1.42
- new net N$25: C10.1, IC4.1, R12.1, R13.2
- new net N$28: C5.+, IC4.4, R12.2
- net +5V: now also C1.+, C2.1, C3.1, D2.C, R10.2, S1.34, S1.35; no longer C5.+, IC4.4
- net GND: now also C10.2, C9.2, LED1.1, LED2.1, R11.1, R13.1; no longer IC3.1, IC4.1
- net N$17: now also IC1.1; no longer IC1.2
- net N$18: now also IC1.2; no longer IC1.1
Routing:
- net +5V: track 40.3 -> 108.9 mm
- net GND: track 317.6 -> 382.6 mm, vias 0 -> 2
- net N$21: track 53.8 -> 0.00 mm
- net N$14: track 47.5 -> 7.80 mm
- net N$17: track 0.00 -> 37.9 mm
- net N$3: track 9.79 -> 38.2 mm, vias 0 -> 2
- net N$28: track 0.00 -> 23.7 mm, vias 0 -> 2
- net N$4: track 5.83 -> 28.8 mm
- net N$13: track 0.00 -> 21.3 mm
- net N$24: track 0.00 -> 17.5 mm
- net N$18: track 51.7 -> 35.3 mm, vias 5 -> 3
- net N$25: track 0.00 -> 13.7 mm
- net N$23: track 0.00 -> 13.7 mm
- net N$16: track 34.6 -> 21.7 mm, vias 1 -> 0
- net N$22: track 0.00 -> 10.6 mm
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
Commit message: Add files via upload
Parts:
- added C11: 100uF, resistor:140CLH-0810
- added Q3, Q4: BC846, BC846B_215:SOT95P230X110-3N
- added R14: 0R, resistor:M1206
- added R15, R17, R19, R20: 4k7, resistor:M1206
- added R16, R18: 47k, resistor:M1206
- C6: value (none) -> 1uF
- C7: value (none) -> 100nF
- C8: value (none) -> 22pF
- R5, R6: value (none) -> 22R
- R7, R8, R9: value (none) -> 51R
- moved D1 82.5 mm to (8.89, 48.3)
- moved Q1 81.6 mm to (12.7, 55.9)
- moved R4 81.6 mm to (12.7, 63.5)
- moved Q2 79.2 mm to (6.35, 55.9)
- moved R3 79.2 mm to (6.35, 63.5)
- moved X2 68.6 mm to (90.2, 80.0), turned to 90 degrees
- moved X3 66.0 mm to (90.2, 90.2), turned to 90 degrees
- moved C6 10.9 mm to (68.6, 11.4)
- moved J1 10.9 mm to (72.4, 0.00)
- moved R5 4.02 mm to (67.3, 35.6)
- moved IC5 3.81 mm to (73.7, 31.8)
- moved R6 3.81 mm to (67.3, 31.8)
Connections:
- new net N$1: Q3.2, R16.2, S1.22
- new net N$21: J2.1, R14.1
- new net N$26: C11.+, S1.28
- new net N$27: Q3.1, R15.2, R16.1
- new net N$30: R15.1, R19.1, R20.1, S1.40
- new net N$32: Q3.3, R17.2, X3.1
- new net N$34: Q4.1, R19.2
- new net N$35: Q4.3, R20.2, S1.23
- new net N$36: Q4.2, R18.2, X2.2
- net GND: now also C11.-, X2.1
- net N$28: now also R17.1, R18.1, X3.2
- net N$5: now also R14.2; no longer J2.1
Routing:
- net N$28: track 23.7 -> 117.5 mm
- net GND: track 382.6 -> 467.2 mm
- net N$35: track 0.00 -> 60.5 mm, vias 0 -> 2
- net N$1: track 0.00 -> 49.4 mm, vias 0 -> 2
- net N$30: track 0.00 -> 31.6 mm
- net N$32: track 0.00 -> 28.3 mm
- net N$15: track 10.6 -> 29.7 mm, vias 0 -> 2
- net N$14: track 7.80 -> 25.9 mm, vias 0 -> 2
- net N$36: track 0.00 -> 17.6 mm
- net N$26: track 0.00 -> 16.9 mm, vias 0 -> 2
- net N$3: track 38.2 -> 50.7 mm
- net N$5: track 16.3 -> 6.27 mm
- net N$21: track 0.00 -> 7.66 mm
- net N$10: track 22.6 -> 30.2 mm
- net N$4: track 28.8 -> 34.3 mm
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
Commit message: Add files via upload
Parts:
- moved C1 1.27 mm to (45.7, 57.1)
- moved R7 1.27 mm to (40.6, 6.35)
- moved R8 1.27 mm to (40.6, 16.5)
- moved R9 1.27 mm to (40.6, 11.4)
Routing:
- net N$30: track 31.6 -> 76.7 mm, vias 0 -> 2
- net N$18: track 35.3 -> 38.4 mm
- net N$15: track 29.7 -> 32.0 mm
- net N$14: track 25.9 -> 27.4 mm
- net N$22: track 10.6 -> 9.38 mm
- net +5V: track 108.9 -> 110.0 mm
- net N$20: track 10.5 -> 9.47 mm

Commit message: Add files via upload
Parts:
- removed D1: 1N4004, diode:DO41-10
- removed R4: (no value), resistor:M1206
- added R21, R23, R24: 4k7, resistor:M1206
- added R22, R25: 47k, resistor:M1206
- added X4, X5: (no value), con-wago-500:W237-102
- C4, C5: value (none) -> 470uF; device resistor:140CLH-0810 -> resistor:140CLH-1010
- C6: device resistor:140CLH-0810 -> resistor:153CLV-0405
- C7: device resistor:140CLH-0810 -> resistor:C0805
- C8: device resistor:C0603 -> resistor:C0805
- IC3: value 317EMP -> 317T; device linear:SOT223 -> linear:TO220H
- J2: value 1 -> Ant GSM
- R1, R2: value (none) -> 3k3
- R3: value (none) -> 4k7
- moved R3 51.2 mm to (53.3, 43.2), turned to 0 degrees
- moved C7 51.1 mm to (83.8, 24.1)
- moved C1 50.8 mm to (95.2, 68.6), turned to 90 degrees
- moved J2 50.3 mm to (121.9, 52.1), turned to 0 degrees
- moved C11 50.0 mm to (105.4, 43.2)
- moved R8 47.4 mm to (85.1, 33.0), turned to 270 degrees
- moved R9 46.0 mm to (81.3, 33.0), turned to 270 degrees
- moved R7 45.5 mm to (77.5, 33.0), turned to 270 degrees
- moved LED1 43.1 mm to (74.9, 68.6)
- moved R1 43.1 mm to (74.9, 63.5)
- moved LED2 41.9 mm to (78.7, 68.6)
- moved R2 41.9 mm to (78.7, 63.5)
- moved C6 40.7 mm to (109.2, 14.0)
- moved J1 40.7 mm to (113.0, 1.27)
- moved C8 38.6 mm to (88.9, 17.8), turned to 270 degrees
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Connections:
- removed net N$11: S1.1
- new net N$31: Q2.2, R22.1, X4.2
- new net N$33: Q2.1, R3.1
- new net N$38: R22.2, R23.1, X5.2
- new net S$3: Q1.2, R25.1, S1.1
- net +5V: now also IC3.2; no longer IC3.4
- net GND: now also C7.2, X4.1; no longer C7.-
- net N$12: now also Q2.3, R21.1
- net N$17: now also C7.1; no longer C7.+
- net N$30: now also R21.2, R24.2, R3.2
- net N$8: now also Q1.3, R23.2, X5.1; no longer Q2.3, R3.1
- net N$9: now also Q1.1, R24.1, R25.2; no longer Q1.3, R4.1
Routing:
- net GND: track 467.4 -> 0.00 mm, vias 2 -> 0
- net N$28: track 117.5 -> 0.00 mm, vias 2 -> 0
- net +5V: track 110.0 -> 0.00 mm
- net N$30: track 76.7 -> 0.00 mm, vias 2 -> 0
- net N$35: track 60.5 -> 0.00 mm, vias 2 -> 0
- net N$3: track 50.7 -> 0.00 mm, vias 2 -> 0
- net N$1: track 49.4 -> 0.00 mm, vias 2 -> 0
- net N$18: track 38.4 -> 0.00 mm, vias 3 -> 0
- net N$17: track 37.9 -> 0.00 mm
- net N$4: track 34.3 -> 0.00 mm
- net N$15: track 32.0 -> 0.00 mm, vias 2 -> 0
- net N$10: track 30.2 -> 0.00 mm
- net N$32: track 28.3 -> 0.00 mm
- net N$14: track 27.4 -> 0.00 mm, vias 2 -> 0
- net N$16: track 21.7 -> 0.00 mm
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Other:
- board size 96.5 x 100 mm -> 160 x 100 mm

Commit message: Add files via upload
Parts:
- moved J2 46.1 mm to (76.2, 57.8)
- moved R25 41.3 mm to (26.0, 55.6)
- moved Q4 36.5 mm to (68.9, 80.3), turned to 90 degrees
- moved R17 36.3 mm to (75.6, 83.8), turned to 0 degrees
- moved R18 36.2 mm to (75.6, 79.7), turned to 0 degrees
- moved Q3 35.6 mm to (69.8, 93.0)
- moved R15 35.3 mm to (58.7, 92.7)
- moved R16 34.9 mm to (64.1, 93.0)
- moved C1 34.9 mm to (61.0, 74.9)
- moved R20 33.1 mm to (73.7, 72.7)
- moved R19 33.1 mm to (68.6, 72.7)
- moved X2 32.2 mm to (88.6, 76.8)
- moved X3 32.2 mm to (88.6, 87.0)
- moved C8 32.1 mm to (56.8, 16.8)
- moved S1 32.1 mm to (49.2, 53.7)
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Routing:
- net GND: track 0.00 -> 460.8 mm, vias 0 -> 3
- net N$28: track 0.00 -> 103.5 mm, vias 0 -> 3
- net +5V: track 0.00 -> 93.8 mm
- net N$30: track 0.00 -> 86.2 mm, vias 0 -> 2
- net N$22: track 0.00 -> 77.3 mm
- net N$3: track 0.00 -> 69.7 mm
- net N$18: track 0.00 -> 62.0 mm
- net N$17: track 0.00 -> 49.3 mm, vias 0 -> 2
- net N$10: track 0.00 -> 47.3 mm
- net N$12: track 0.00 -> 41.5 mm, vias 0 -> 2
- net N$16: track 0.00 -> 41.0 mm, vias 0 -> 1
- net N$4: track 0.00 -> 39.8 mm
- net N$14: track 0.00 -> 37.6 mm
- net N$20: track 0.00 -> 32.5 mm
- net N$13: track 0.00 -> 30.1 mm
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Other:
- board size 160 x 100 mm -> 95.2 x 100 mm

Commit message: Add files via upload
Parts:
- moved R16 27.3 mm to (76.2, 68.6)
- moved Q3 26.7 mm to (80.6, 68.6)
- moved R15 26.6 mm to (71.8, 69.5), turned to 0 degrees
- moved R8 14.5 mm to (55.2, 29.2)
- moved IC2 12.9 mm to (65.1, 30.2), turned to 0 degrees
- moved C6 8.98 mm to (86.4, 28.6), turned to 270 degrees
- moved R19 8.31 mm to (76.8, 73.7), turned to 0 degrees
- moved IC5 8.25 mm to (76.8, 24.8)
- moved Q4 8.14 mm to (76.5, 77.5), turned to 180 degrees
- moved R9 7.03 mm to (59.1, 29.2)
- moved D2 6.03 mm to (53.7, 74.3)
- moved C2 4.84 mm to (53.0, 63.8), turned to 180 degrees
- moved R17 4.42 mm to (71.4, 85.4)
- moved R18 4.24 mm to (71.4, 80.6)
- moved C3 3.70 mm to (56.8, 63.8), turned to 0 degrees
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Routing:
- net N$22: track 77.3 -> 23.2 mm
- net N$35: track 0.00 -> 47.7 mm, vias 0 -> 2
- net N$1: track 5.06 -> 43.5 mm, vias 0 -> 2
- net N$15: track 10.1 -> 35.9 mm
- net N$18: track 62.0 -> 39.0 mm, vias 0 -> 2
- net N$32: track 13.5 -> 36.2 mm, vias 0 -> 1
- net N$29: track 0.00 -> 18.1 mm
- net GND: track 460.8 -> 475.8 mm, vias 3 -> 10
- net N$30: track 86.2 -> 71.7 mm, vias 2 -> 3
- net N$10: track 47.3 -> 61.4 mm
- net N$14: track 37.6 -> 28.9 mm, vias 0 -> 2
- net N$3: track 69.7 -> 77.5 mm
- net N$36: track 25.9 -> 19.8 mm, vias 0 -> 1
- net N$33: track 11.1 -> 5.10 mm
- net N$24: track 11.7 -> 6.09 mm
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
Commit message: Add files via upload
Parts:
- moved J1 10.6 mm to (77.8, 1.91)
- moved C6 5.79 mm to (80.6, 29.5), turned to 180 degrees
- moved C3 4.96 mm to (53.0, 67.0), turned to 180 degrees
- moved IC5 4.84 mm to (74.9, 29.2), turned to 90 degrees
- moved C9 4.49 mm to (31.4, 82.5)
- moved C11 2.86 mm to (81.9, 47.3)
- moved R22 2.84 mm to (15.9, 54.0)
- moved D2 2.25 mm to (52.1, 75.9)
- moved LED2 1.90 mm to (47.9, 69.5)
- moved R2 1.90 mm to (47.9, 64.5)
- moved R10 1.00 mm to (32.4, 85.4), turned to 0 degrees
- moved C1 0.95 mm to (60.0, 74.9)
- moved LED1 0.95 mm to (45.1, 69.5)
- moved R1 0.95 mm to (45.1, 64.5)
- moved Q1 0.95 mm to (21.0, 55.9)
Connections:
- net N$10: now also IC5.1; no longer IC5.2
- net N$4: now also IC5.2; no longer IC5.1
Routing:
- net GND: track 475.8 -> 528.6 mm, vias 10 -> 11
- net N$11: track 0.00 -> 27.3 mm
- net N$10: track 61.4 -> 40.8 mm
- net N$3: track 77.5 -> 61.9 mm, vias 0 -> 2
- net N$37: track 0.00 -> 4.76 mm
- net N$28: track 103.8 -> 99.8 mm
- net N$16: track 41.0 -> 44.9 mm
- net N$26: track 28.8 -> 26.0 mm
- net N$15: track 35.9 -> 33.3 mm
- net +5V: track 90.6 -> 88.5 mm
- net N$19: track 15.2 -> 13.2 mm
- net N$12: track 40.5 -> 42.3 mm, vias 2 -> 0
- net N$14: track 28.9 -> 30.8 mm
- net N$20: track 28.6 -> 30.1 mm
- net N$23: track 7.41 -> 5.94 mm
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
Commit message: Add files via upload
Parts:
- moved C1 3.13 mm to (57.1, 73.7), turned to 0 degrees
- moved D2 1.80 mm to (50.8, 77.2)
- moved R22 1.71 mm to (14.3, 53.3), turned to 180 degrees
- moved C2 1.27 mm to (51.8, 63.8)
- moved C3 1.27 mm to (51.8, 67.0)
- moved R23 0.63 mm to (14.3, 46.7)
Routing:
- net GND: track 528.6 -> 521.6 mm
- net +5V: track 88.5 -> 83.4 mm
- net N$37: track 4.76 -> 0.00 mm
- net N$38: track 19.1 -> 20.6 mm, vias 0 -> 1
- net N$31: track 21.6 -> 22.9 mm
- net N$16: track 44.9 -> 43.8 mm
- net N$30: track 70.4 -> 71.3 mm
